File: pcb/evaluationBoard/GPS.sch (KiCad schematic (older format))
At the start: 0 parts

Commit message: added modules
Parts:
- added IC?: ATGM336H-5N31, ATGM336H5N31, symbol RF_JLC:ATGM336H-5N31
Changed lines of the file:
@@
 $Descr A4 11693 8268
 encoding utf-8
-Sheet 1 4
+Sheet 4 7
 Title ""
 Date ""
@@
 Comment4 ""
 $EndDescr
+$Comp
+L RF_JLC:ATGM336H-5N31 IC?
+U 1 1 6027EAEB
+P 4600 3200
+F 0 "IC?" H 5350 3465 50  0000 C CNN
+F 1 "ATGM336H-5N31" H 5350 3374 50  0000 C CNN
+F 2 "ATGM336H5N31" H 5950 3300 50  0001 L CNN
+F 3 "https://datasheet.lcsc.com/szlcsc/ZHONGKEWEI-ATGM336H-5N31_C90770.pdf" H 5950 3200 50  0001 L CNN
+F 4 "GSM & GPRS & GPS Modules 9.7X10.1mm RoHS" H 5950 3100 50  0001 L CNN "Description"
+F 5 "2.6" H 5950 3000 50  0001 L CNN "Height"
+F 6 "ZHONGKEWEI" H 5950 2900 50  0001 L CNN "Manufacturer_Name"
+F 7 "ATGM336H-5N31" H 5950 2800 50  0001 L CNN "Manufacturer_Part_Number"
+F 8 "C90770" H 4600 3200 50  0001 C CNN "LCSC"
+	1    4600 3200
+	1    0    0    -1
+$EndComp
 $EndSCHEMATC
