File: pcb/evaluationBoard/dsp.sch (KiCad schematic (older format))
At the start: 8 parts

Commit message: wip
Parts:
- removed C?: 47n, Capacitor_SMD:C_0402_1005Metric, symbol Capacitor_JLC:47n
- removed C?: 47uF, Capacitor_SMD:C_1206_3216Metric, symbol Capacitor_JLC:47uF
- removed R?: 2.7k, Resistor_SMD:R_0402_1005Metric, symbol Resistor_JLC:2.7k
- added AT1, AT2: LM386MX-1_NOPB, SOIC127P600X175-8N, symbol Power-Drivers_JLC:LM386MX-1_NOPB
- added C1, C6, C7, C8: 33p, Capacitor_SMD:C_0402_1005Metric, symbol Capacitor_JLC:33p
- added C10, C12, C14: 10u, Capacitor_SMD:C_0805_2012Metric, symbol Capacitor_JLC:10u
- added C15, C16, C2, C21, C22, C23, C24, C3, C33, C34, C4, C5: 100n, Capacitor_SMD:C_0402_1005Metric, symbol Capacitor_JLC:100n
- added C17, C18: 47uF, Capacitor_SMD:C_1206_3216Metric, symbol Capacitor_JLC:47uF
- added C19, C20: 4.7n, Capacitor_SMD:C_0402_1005Metric, symbol Capacitor_JLC:4.7n
- added C25, C26, C31, C32: NA_C, Capacitor_SMD:C_0805_2012Metric_Pad1.18x1.45mm_HandSolder, symbol Capacitor_JLC:NA_C
- added C27, C28: 47n, Capacitor_SMD:C_0402_1005Metric, symbol Capacitor_JLC:47n
- added C29, C30: 220uF_E, Capacitor_SMD:CP_Elec_10x10, symbol Capacitor_JLC:220uF_E
- added IC2: TLV320AIC3254IRHBT, SamacSys_Parts:QFN50P500X500X100-33N-D, symbol Misc_JLC:TLV320AIC3254IRHBT
- added R1, R10, R2, R3, R4, R8, R9: 22, Resistor_SMD:R_0402_1005Metric, symbol Resistor_JLC:22
- added R12, R14, R15, R5: 1k, Resistor_SMD:R_0402_1005Metric, symbol Resistor_JLC:1k
- added R13: 2.7k, Resistor_SMD:R_0402_1005Metric, symbol Resistor_JLC:2.7k
- added R16, R17: NA_R, Resistor_SMD:R_0805_2012Metric_Pad1.20x1.40mm_HandSolder, symbol Resistor_JLC:NA_R
- added R18, R19, R7: 10, Resistor_SMD:R_0603_1608Metric, symbol Resistor_JLC:10
- gave numbers to parts that had none: 5
Connections:
- net MICBIAS: now reaches R11.1
- net MICBIAS: now also IC2.19 (MICBIAS), R13.1, R5.1
- net -IN1_L: now reaches R11.2
- net -IN1_L: now also C2.2
- net +3V3: now reaches C13.1
- net +3V3: now also C11.1, C9.1, IC2.26 (LDOIN), IC2.30 (LDO_SELECT), IC2.6 (IOVDD)
- net GND: now reaches C13.2
- net GND: now also C11.2, C9.2, R6.2, AT1.4 (GND), AT2.4 (GND), C1.2, C10.2, C12.2, C14.2, C19.2, C20.2, C22.2, C24.2, C27.2, C28.2, C31.1, C32.1, C33.1, C34.1, C6.2, C7.2, C8.2, IC2.12 (SPI_SELECT), IC2.17 (AVSS), IC2.28 (DVSS), IC2.33 (GND), IC2.7 (IOVSS), R12.2
- net -IN2_R: now reaches R6.1
- net -IN2_R: now also C5.2
- new net: IC2.1 (MCLK), R7.1
- new net: IC2.10 (SDA/MOSI), R10.1
- new net: IC2.11 (MISO/MFP4), R4.1
- new net: C1.1, C2.1, IC2.13 (IN1_L)
- new net: C3.1, C6.1, IC2.14 (IN1_R)
- new net: C4.1, C7.1, IC2.15 (IN2_L)
- new net: C5.1, C8.1, IC2.16 (IN2_R)
- new net: C10.1, C12.1, C14.1, IC2.18 (REF), IC2.24 (AVDD), IC2.29 (DVDD)
- new net: IC2.2 (BCLK), R1.1
- new net: C15.2, IC2.20 (IN3_L)
- new net: C16.2, IC2.21 (IN3_R)
- new net: C17.2, IC2.25 (HPL)
- new net: C18.2, IC2.27 (HPR)
- new net: IC2.3 (WCLK), R8.1
- new net: IC2.4 (DIN/MFP1), R2.1
- new net: IC2.5 (DOUT/MFP2), R9.1
- new net: IC2.9 (SCL/~SS), R3.1
- new net: AT1.1 (GAIN_1), R16.2
- new net: AT1.2 (-INPUT), C21.1
- new net: AT1.3 (+INPUT), C22.1
- new net: AT1.5 (VOUT), C29.1, R18.1
- new net: AT1.7 (BYPASS), C31.2
- new net: AT1.8 (GAIN_2), C25.1
- new net: C19.1, C21.2, R14.1
- new net: C25.2, R16.1
- new net: C27.1, R18.2
- new net: AT2.1 (GAIN_1), R17.2
- new net: AT2.2 (-INPUT), C23.1
- new net: AT2.3 (+INPUT), C24.1
- new net: AT2.5 (VOUT), C30.1, R19.1
- new net: AT2.7 (BYPASS), C32.2
- new net: AT2.8 (GAIN_2), C26.1
- new net: C20.1, C23.2, R15.1
- new net: C26.2, R17.1
- new net: C28.1, R19.2
- new net -HPL: C17.1
- new net -HPR: C18.1
- new net -IN1_R: C3.2, R12.1
- new net -IN2_L: C4.2, R5.2
- new net -LOL: C29.2
- new net -LOR: C30.2
- new net BCLK: R1.2
- new net DIN: R2.2
- new net DOUT: R9.2
- new net GPIO: IC2.32 (GPIO/MFP5)
- new net LOL: IC2.22 (LOL), R14.2
- new net LOR: IC2.23 (LOR), R15.2
- new net MCLK: R7.2
- new net MIC+: C16.1, IC2.8 (SCLK/MFP3), R13.2
- new net MIC-: C15.1
- new net MISO: R4.2
- new net SCL: R3.2
- new net SDA: R10.2
- new net VDC: AT1.6 (VS), AT2.6 (VS), C33.2, C34.2
- new net WCLK: R8.2
- new net ~RESET: IC2.31 (~RESET)
Other:
- moved on the sheet: C11, C13, C9, R11, R6
