File: pcb/evaluationBoard/power.sch (KiCad schematic (older format))
At the start: 26 parts, among them IC2 TPS5430DDAR, IC3 TPS54331DR

Commit message: updated design
Parts:
- removed L1: 15uH, SWRB1204S150MT, symbol Inductor_JLC:15uH
- added L?: 15uH, SamacSys_Parts:SWRB1204S150MT, symbol Inductor_JLC:15uH
- added L?: 6.8uH, SamacSys_Parts:INDPM6060X450N, symbol Inductor_JLC:6.8uH
- renumbered C1 to C?, C3 to C?, C2 to C?, C5 to C?, C6 to C?, C7 to C?, C9 to C?, C11 to C?, C10 to C?, C4 to C?, C8 to C?, C12 to C?, D1 to D?, D2 to D?, IC2 to IC?, IC3 to IC?, L2 to L?, R1 to R?, R2 to R?, R3 to R?, R4 to R?, R6 to R?, R7 to R?, R8 to R?, R5 to R?
Connections:
- net +3V3: now also L?.2
- net at C?.1, D?.1, IC?.8 (PH): now also L?.1 (x2)
- net at L?.1: now also L?.2
Other:
- moved on the sheet: L?

Commit message: wip
Parts:
- gave numbers to parts that had none: 27
